File: hardware/usb-can-adapter/usb-can-adapter.kicad_pcb (KiCad board)
At the start: 2 copper layers, 40 x 20 mm, 42 parts, among them J1 SWD, J2 USB_C_Receptacle_USB2.0_16P, J3 Conn_01x03, J4 Conn_01x02, Q1 AO3401A, Q2 2N7002, SW1 SW_Push, U1 STM32G431CBTx, U2 AP2112K-3.3, U3 USBLC6-2SC6, U4 SN65HVD230, Y1 24MHz

Commit message: feat(adapter): enlarge pcb to 50x25, place mcu block
Resize outline for easier hand soldering, place usb, ldo, mcu, crystal and decoupling capacitors.
Parts:
- moved U3 78.9 mm to (111.7, 110.3)
- moved R5 77.4 mm to (111.8, 113.3)
- moved R4 77.3 mm to (111.8, 107.2)
- moved Y1 71.3 mm to (134.1, 113.2), turned to 180 degrees
- moved U2 70.9 mm to (120.2, 105.5)
- moved C1 65.7 mm to (112.5, 118.6)
- moved U1 64.6 mm to (126.4, 112.1), turned to 180 degrees
- moved C12 64.0 mm to (116.0, 105.0)
- moved C7 61.7 mm to (119.1, 109.9)
- moved C2 59.1 mm to (116.0, 107.3)
- moved C4 59.1 mm to (116.9, 118.7)
- moved C10 58.6 mm to (122.3, 119.2)
- moved C8 54.9 mm to (127.7, 118.4)
- moved C14 52.1 mm to (134.7, 116.3)
- moved C11 51.5 mm to (128.2, 105.7)
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Other:
- board size 40 x 20 mm -> 50 x 25 mm
